Commit message: Fix station collada mesh, create smaller station mesh, add stone mesh, create rotation script

File: urdf/gravity_decor.urdf (robot description, URDF)
Before this commit: robot gravity_description, 1 links, 0 joints
Links:
- link obstacle_base: geometry visual mesh filename=package://gravity_description/meshes/station.dae
